File: BBNL_PDU_Protector/BBNL_PDU_Protector.kicad_sch (KiCad schematic)
At the start: 20 parts, among them J1 1720796, J2 1708381

Commit message: second commit
Parts:
- H1, H2, H3, H4, H5: footprint MountingHole:MountingHole_4mm_Pad_TopBottom -> MountingHole:MountingHole_3mm_Pad_TopBottom
Connections:
- net Earth: no longer H1.1, H2.1
- no-connect marks 0 -> 3
Other:
- moved on the sheet: H1, H2
Changed lines of the file:
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@@
   (junction (at 102.87 87.63) (diameter 0) (color 0 0 0 0)
   )
+  (junction (at 189.23 91.44) (diameter 0) (color 0 0 0 0)
+  )
   (junction (at 186.69 91.44) (diameter 0) (color 0 0 0 0)
   )
-  (junction (at 175.26 91.44) (diameter 0) (color 0 0 0 0)
-  )
   (junction (at 82.55 74.93) (diameter 0) (color 0 0 0 0)
   )
@@
   (junction (at 82.55 85.09) (diameter 0) (color 0 0 0 0)
   )
+  (no_connect (at 69.85 77.47))
+  (no_connect (at 176.53 73.66))
+  (no_connect (at 181.61 73.66))
   (wire (pts (xy 181.61 91.44) (xy 186.69 91.44))
     (stroke (width 0) (type default) (color 0 0 0 0))
@@
     (stroke (width 0) (type default) (color 0 0 0 0))
   )
+  (wire (pts (xy 189.23 91.44) (xy 191.77 91.44))
+    (stroke (width 0) (type default) (color 0 0 0 0))
+  )
   (wire (pts (xy 130.81 82.55) (xy 130.81 87.63))
     (stroke (width 0) (type default) (color 0 0 0 0))
@@
     (stroke (width 0) (type default) (color 0 0 0 0))
   )
-  (wire (pts (xy 175.26 90.17) (xy 175.26 91.44))
-    (stroke (width 0) (type default) (color 0 0 0 0))
-  )
   (wire (pts (xy 111.76 77.47) (xy 111.76 74.93))
     (stroke (width 0) (type default) (color 0 0 0 0))
@@
   )
   (wire (pts (xy 80.01 77.47) (xy 82.55 77.47))
-    (stroke (width 0) (type default) (color 0 0 0 0))
-  )
-  (wire (pts (xy 181.61 90.17) (xy 181.61 91.44))
     (stroke (width 0) (type default) (color 0 0 0 0))
   )
@@
       (effects (font (size 1.27 1.27)) (justify right) hide)
     )
-    (property "Footprint" "MountingHole:MountingHole_4mm_Pad_TopBottom" (id 2) (at 181.61 96.52 0)
+    (property "Footprint" "MountingHole:MountingHole_3mm_Pad_TopBottom" (id 2) (at 181.61 96.52 0)
       (effects (font (size 1.27 1.27)) hide)
     )
@@
     (pin "2")
   )
-  (symbol (lib_id "Mechanical:MountingHole_Pad") (at 181.61 87.63 0) (unit 1)
-    (in_bom yes) (on_board yes)
-    (property "Reference" "H2" (id 0) (at 180.34 82.55 0)
-      (effects (font (size 1.27 1.27)) (justify left))
-    )
-    (property "Value" "MountingHole_Pad" (id 1) (at 184.15 87.6299 0)
-      (effects (font (size 1.27 1.27)) (justify left) hide)
-    )
-    (property "Footprint" "MountingHole:MountingHole_4mm_Pad_TopBottom" (id 2) (at 181.61 87.63 0)
-      (effects (font (size 1.27 1.27)) hide)
-    )
-    (property "Datasheet" "~" (id 3) (at 181.61 87.63 0)
+  (symbol (lib_id "Mechanical:MountingHole_Pad") (at 181.61 71.12 0) (unit 1)
+    (in_bom yes) (on_board yes)
+    (property "Reference" "H2" (id 0) (at 180.34 66.04 0)
+      (effects (font (size 1.27 1.27)) (justify left))
+    )
+    (property "Value" "MountingHole_Pad" (id 1) (at 184.15 71.1199 0)
+      (effects (font (size 1.27 1.27)) (justify left) hide)
+    )
+    (property "Footprint" "MountingHole:MountingHole_3mm_Pad_TopBottom" (id 2) (at 181.61 71.12 0)
+      (effects (font (size 1.27 1.27)) hide)
+    )
+    (property "Datasheet" "~" (id 3) (at 181.61 71.12 0)
       (effects (font (size 1.27 1.27)) hide)
     )
@@
     (pin "2")
   )
-  (symbol (lib_id "Mechanical:MountingHole_Pad") (at 175.26 87.63 0) (unit 1)
-    (in_bom yes) (on_board yes)
-    (property "Reference" "H1" (id 0) (at 173.99 82.55 0)
-      (effects (font (size 1.27 1.27)) (justify left))
-    )
-    (property "Value" "MountingHole_Pad" (id 1) (at 177.8 87.6299 0)
-      (effects (font (size 1.27 1.27)) (justify left) hide)
-    )
-    (property "Footprint" "MountingHole:MountingHole_4mm_Pad_TopBottom" (id 2) (at 175.26 87.63 0)
-      (effects (font (size 1.27 1.27)) hide)
-    )
-    (property "Datasheet" "~" (id 3) (at 175.26 87.63 0)
+  (symbol (lib_id "Mechanical:MountingHole_Pad") (at 176.53 71.12 0) (unit 1)
+    (in_bom yes) (on_board yes)
+    (property "Reference" "H1" (id 0) (at 175.26 66.04 0)
+      (effects (font (size 1.27 1.27)) (justify left))
+    )
+    (property "Value" "MountingHole_Pad" (id 1) (at 179.07 71.1199 0)
+      (effects (font (size 1.27 1.27)) (justify left) hide)
+    )
+    (property "Footprint" "MountingHole:MountingHole_3mm_Pad_TopBottom" (id 2) (at 176.53 71.12 0)
+      (effects (font (size 1.27 1.27)) hide)
+    )
+    (property "Datasheet" "~" (id 3) (at 176.53 71.12 0)
       (effects (font (size 1.27 1.27)) hide)
     )
@@
     (pin "1")
     (pin "3")
+  )
+  (symbol (lib_id "power:PWR_FLAG") (at 191.77 91.44 270) (unit 1)
+    (in_bom yes) (on_board yes) (fields_autoplaced)
+    (property "Reference" "#FLG0101" (id 0) (at 193.675 91.44 0)
+      (effects (font (size 1.27 1.27)) hide)
+    )
+    (property "Value" "PWR_FLAG" (id 1) (at 195.58 91.4399 90)
+      (effects (font (size 1.27 1.27)) (justify left))
+    )
+    (property "Footprint" "" (id 2) (at 191.77 91.44 0)
+      (effects (font (size 1.27 1.27)) hide)
+    )
+    (property "Datasheet" "~" (id 3) (at 191.77 91.44 0)
+      (effects (font (size 1.27 1.27)) hide)
+    )
+    (pin "1")
   )
   (symbol (lib_id "Device:L") (at 118.11 74.93 90) (unit 1)
@@
       (effects (font (size 1.27 1.27)) (justify right) hide)
     )
-    (property "Footprint" "MountingHole:MountingHole_4mm_Pad_TopBottom" (id 2) (at 175.26 96.52 0)
+    (property "Footprint" "MountingHole:MountingHole_3mm_Pad_TopBottom" (id 2) (at 175.26 96.52 0)
       (effects (font (size 1.27 1.27)) hide)
     )
@@
       (effects (font (size 1.27 1.27)) (justify left) hide)
     )
-    (property "Footprint" "MountingHole:MountingHole_4mm_Pad_TopBottom" (id 2) (at 186.69 87.63 0)
+    (property "Footprint" "MountingHole:MountingHole_3mm_Pad_TopBottom" (id 2) (at 186.69 87.63 0)
       (effects (font (size 1.27 1.27)) hide)
     )
@@
   )
   (symbol_instances
+    (path "/8c8a6b4b-8d32-4980-a58e-b96d540ef4cf"
+      (reference "#FLG0101") (unit 1) (value "PWR_FLAG") (footprint "")
+    )
     (path "/ca0d4fed-6035-48b4-b0d8-b6eaa9c8f16b"
       (reference "#PWR0101") (unit 1) (value "Earth") (footprint "")
@@
     )
     (path "/77fce35a-c36c-41a9-8577-ebeaf1cf3828"
-      (reference "H1") (unit 1) (value "MountingHole_Pad") (footprint "MountingHole:MountingHole_4mm_Pad_TopBottom")
+      (reference "H1") (unit 1) (value "MountingHole_Pad") (footprint "MountingHole:MountingHole_3mm_Pad_TopBottom")
     )
     (path "/3ee50426-7932-4659-9f19-80824ea5f05a"
-      (reference "H2") (unit 1) (value "MountingHole_Pad") (footprint "MountingHole:MountingHole_4mm_Pad_TopBottom")
+      (reference "H2") (unit 1) (value "MountingHole_Pad") (footprint "MountingHole:MountingHole_3mm_Pad_TopBottom")
     )
     (path "/b5819bf1-4e57-40e0-afe7-6d104717d81a"
-      (reference "H3") (unit 1) (value "MountingHole_Pad") (footprint "MountingHole:MountingHole_4mm_Pad_TopBottom")
+      (reference "H3") (unit 1) (value "MountingHole_Pad") (footprint "MountingHole:MountingHole_3mm_Pad_TopBottom")
     )
     (path "/02bc88a7-fbda-4ab5-9292-f0682fa275b2"
-      (reference "H4") (unit 1) (value "MountingHole_Pad") (footprint "MountingHole:MountingHole_4mm_Pad_TopBottom")
+      (reference "H4") (unit 1) (value "MountingHole_Pad") (footprint "MountingHole:MountingHole_3mm_Pad_TopBottom")
     )
     (path "/d1c5aed9-97e8-4287-a86a-42101f0e9ca7"
-      (reference "H5") (unit 1) (value "MountingHole_Pad") (footprint "MountingHole:MountingHole_4mm_Pad_TopBottom")
+      (reference "H5") (unit 1) (value "MountingHole_Pad") (footprint "MountingHole:MountingHole_3mm_Pad_TopBottom")
     )
     (path "/63b4b4d1-394b-4d8f-b82e-e3a60856e1a5"

Commit message: 27.06.24 commit
Connections:
- no-connect marks 3 -> 2
Changed lines of the file:
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@@
   (junction (at 82.55 85.09) (diameter 0) (color 0 0 0 0)
   )
-  (no_connect (at 69.85 77.47))
   (no_connect (at 176.53 73.66))
   (no_connect (at 181.61 73.66))
