File: JT_CCU_AC_Surge_Protection_Board/JT_CCU_AC_Surge_Protection_Board/JT_CCU_AC_Surge_Protection_Board.kicad_sch (KiCad schematic)
At the start: 14 parts, among them J1 Grid Surge Input, J2 Grid Surge Out

Commit message: 27.06.24 commit
Parts:
- removed J1: Grid Surge Input, symbol Connector:Conn_01x03_Male
- removed J2: Grid Surge Out, symbol Connector:Conn_01x03_Male
- added J1: L, ACSPD:quickfit_PCB, symbol Connector:Conn_01x01_Female
- added J2: E, ACSPD:quickfit_PCB, symbol Connector:Conn_01x01_Female
- added J3: N, ACSPD:quickfit_PCB, symbol Connector:Conn_01x01_Female
- added J4: L, ACSPD:Out_conn, symbol Connector:Conn_01x01_Female
- added J5: E, ACSPD:Out_conn, symbol Connector:Conn_01x01_Female
- added J6: N, ACSPD:Out_conn, symbol Connector:Conn_01x01_Female
- added L1, L2: INDUCTOR, ACSPD:EE16-SS-1, symbol pspice:INDUCTOR
- F1, F2: footprint (none) -> ACSPD:Fuse
- GD1, GD2: footprint (none) -> ACSPD:GD Tube
- H1, H2, H3, H4: footprint (none) -> ACSPD:CCU_GND_PT
- RV1, RV2: footprint (none) -> MOV-20D391KKTR:MOV20D391KKTR
- RV3, RV4: footprint (none) -> GMOV-20D251K:GMOV20D251K
Connections:
- net Earth: now also J2.1 (Pin_1), J5.1 (Pin_1)
- net at F2.2, RV2.2: now also L2.2; no longer RV4.2
- net at F1.2, RV1.1: now also L1.1; no longer RV3.1
- net at F2.1: now also J3.1 (Pin_1)
- net at F1.1: now also J1.1 (Pin_1)
- new net: J4.1 (Pin_1), L1.2, RV3.1
- new net: J6.1 (Pin_1), L2.1, RV4.2
