File: JT_CCU_AC_Surge_Protection_Board/JT_CCU_AC_Surge_Protection_Board/JT_CCU_AC_Surge_Protection_Board.kicad_pcb (KiCad board)
At the start: 2 copper layers, 103.4 x 68.8 mm, 0 parts

Commit message: 27.06.24 commit
Parts:
- added F1: Fuse, ACSPD:Fuse, F.Cu at (106.0, 77.5)
- added F2: Fuse, ACSPD:Fuse, F.Cu at (106.0, 89.1)
- added GD1: GDT_2Pin, ACSPD:GD Tube, F.Cu at (131.3, 57.6)
- added GD2: GDT_2Pin, ACSPD:GD Tube, F.Cu at (131.2, 109.0)
- added H1: MountingHole_Pad, ACSPD:CCU_GND_PT, F.Cu at (75.3, 56.2)
- added H2: MountingHole_Pad, ACSPD:CCU_GND_PT, F.Cu at (75.3, 112.8)
- added H3: MountingHole_Pad, ACSPD:CCU_GND_PT, F.Cu at (168.5, 56.2)
- added H4: MountingHole_Pad, ACSPD:CCU_GND_PT, F.Cu at (168.5, 112.8)
- added J1: L, ACSPD:quickfit_PCB, F.Cu at (74.4, 69.5)
- added J2: E, ACSPD:quickfit_PCB, F.Cu at (74.4, 100.5)
- added J3: N, ACSPD:quickfit_PCB, F.Cu at (74.4, 85.0)
- added J4: L, ACSPD:Out_conn, F.Cu at (168.3, 70.5)
- added J5: E, ACSPD:Out_conn, F.Cu at (168.3, 104.8)
- added J6: N, ACSPD:Out_conn, F.Cu at (168.3, 88.6)
- added L1: INDUCTOR, ACSPD:EE16-SS-1, F.Cu at (140.6, 73.0)
- added L2: INDUCTOR, ACSPD:EE16-SS-1, F.Cu at (140.1, 93.4)
- added RV1: Varistor, MOV-20D391KKTR:MOV20D391KKTR, F.Cu at (111.0, 67.0)
- added RV2: Varistor, MOV-20D391KKTR:MOV20D391KKTR, F.Cu at (121.3, 99.1)
- added RV3: GMOC, GMOV-20D251K:GMOV20D251K, F.Cu at (156.1, 71.5)
- added RV4: GMOC, GMOV-20D251K:GMOV20D251K, F.Cu at (156.3, 104.2)
Routing:
- net Net-(F2-Pad2): track 0.00 -> 38.9 mm
- net Net-(J6-Pad1): track 0.00 -> 37.3 mm
- net Net-(F1-Pad2): track 0.00 -> 37.2 mm
- net Net-(J4-Pad1): track 0.00 -> 32.4 mm
- net Net-(F1-Pad1): track 0.00 -> 24.8 mm
- net Net-(GD1-Pad3): track 0.00 -> 21.5 mm
- net Net-(GD2-Pad1): track 0.00 -> 21.3 mm
- net Net-(F2-Pad1): track 0.00 -> 18.3 mm
- added copper zone on F.Cu, net Earth

Commit message: 27.06.24 commit
Parts:
- moved RV2 13.4 mm to (113.7, 110.1)
- moved RV1 10.2 mm to (106.3, 57.9)
- moved GD1 5.28 mm to (136.4, 56.3), turned to 180 degrees
- moved F1 3.10 mm to (106.0, 74.4)
- moved GD2 2.25 mm to (133.1, 110.2), turned to 0 degrees
- moved F2 2.20 mm to (106.1, 91.3)
Routing:
- net Net-(F1-Pad2): track 37.2 -> 53.0 mm
- net Net-(F2-Pad2): track 38.9 -> 54.2 mm
- net Net-(GD2-Pad1): track 21.3 -> 12.2 mm
- net Net-(GD1-Pad3): track 21.5 -> 13.5 mm
- net Net-(F1-Pad1): track 24.8 -> 20.1 mm
- net Net-(J6-Pad1): track 37.3 -> 35.1 mm
- net Net-(F2-Pad1): track 18.3 -> 19.4 mm
